File: game-boy-pico-link-board.kicad_pcb (KiCad board)
At the start: 2 copper layers, 85.5 x 26 mm, 6 parts, among them J1 GBA_Link, J2 DMG_Link, J3 Breakout, SW1 SW_SPDT, U1 Pico_Reduced, U2 BOB-12009

Commit message: Minor rerouting
Update design to v1.6
Routing:
- net /PSC: track 74.2 -> 77.7 mm
Other:
- board text added: "version 1.6 2023"
- board text removed: "version 1.5 2023"
Changed lines of the file:
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@@
     (effects (font (size 1 1) (thickness 0.15)) (justify left bottom mirror))
   )
-  (gr_text "version 1.5\n2023" (at 117.71 95.4 180) (layer "B.SilkS")
+  (gr_text "version 1.6\n2023" (at 117.71 95.4 180) (layer "B.SilkS")
     (effects (font (size 1 1) (thickness 0.25) bold) (justify mirror))
   )
@@
   (segment (start 128.935 85.4789) (end 129.3081 85.852) (width 0.5) (layer "B.Cu") (net 9))
   (segment (start 129.3081 85.852) (end 130.81 85.852) (width 0.5) (layer "B.Cu") (net 9))
-  (segment (start 72.9 102.36) (end 73.74 101.52) (width 0.5) (layer "F.Cu") (net 10))
-  (segment (start 72.9 104.775) (end 72.9 102.36) (width 0.5) (layer "F.Cu") (net 10))
-  (segment (start 76.0722 101.52) (end 85.1611 92.4311) (width 0.5) (layer "F.Cu") (net 10))
-  (segment (start 85.1611 92.4311) (end 137.5369 92.4311) (width 0.5) (layer "F.Cu") (net 10))
-  (segment (start 137.5369 92.4311) (end 139.67 90.298) (width 0.5) (layer "F.Cu") (net 10))
-  (segment (start 73.74 101.52) (end 76.0722 101.52) (width 0.5) (layer "F.Cu") (net 10))
+  (segment (start 126.511608 94.6156) (end 135.7624 94.6156) (width 0.5) (layer "F.Cu") (net 10))
+  (segment (start 135.7624 94.6156) (end 138.176 92.202) (width 0.5) (layer "F.Cu") (net 10))
+  (segment (start 72.9 102.868) (end 73.406 102.362) (width 0.5) (layer "F.Cu") (net 10))
+  (segment (start 124.5576 96.569608) (end 126.511608 94.6156) (width 0.5) (layer "F.Cu") (net 10))
+  (segment (start 123.952 102.362) (end 124.5576 101.7564) (width 0.5) (layer "F.Cu") (net 10))
+  (segment (start 72.9 104.775) (end 72.9 102.868) (width 0.5) (layer "F.Cu") (net 10))
+  (segment (start 138.176 92.202) (end 139.117308 92.202) (width 0.5) (layer "F.Cu") (net 10))
+  (segment (start 139.117308 92.202) (end 139.67 91.649308) (width 0.5) (layer "F.Cu") (net 10))
+  (segment (start 73.406 102.362) (end 123.952 102.362) (width 0.5) (layer "F.Cu") (net 10))
+  (segment (start 124.5576 101.7564) (end 124.5576 96.569608) (width 0.5) (layer "F.Cu") (net 10))
+  (segment (start 139.67 91.649308) (end 139.67 90.298) (width 0.5) (layer "F.Cu") (net 10))
   (segment (start 123.79 99.21) (end 126.5 96.5) (width 0.5) (layer "B.Cu") (net 11))
   (segment (start 132.3 96.5) (end 137.13 91.67) (width 0.5) (layer "B.Cu") (net 11))
